Commit message: chore: sync friday_ros2 from holiday
GitOrigin-RevId: 0518e92011ca8333abcd0246a3dce5f44badc0ef

File: friday_description/urdf/FM26B.urdf (robot description, URDF)
Before this commit: robot FM26B, 90 links, 89 joints
Links:
- link left_arm_7: geometry collision mesh filename=package://friday_description/meshes/FM26B/visual/left_arm_7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; collision mesh filename=package://friday_description/meshes/FM26B/visual/left_wrist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
- link left_hand_1_2: geometry collision mesh filename=package://friday_description/meshes/FM26B/visual/left_hand_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; collision mesh filename=package://friday_description/meshes/FM26B/visual/tactile_th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
- link left_hand_1_3: geometry collision mesh filename=package://friday_description/meshes/FM26B/visual/left_hand_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; collision mesh filename=package://friday_description/meshes/FM26B/visual/tactile_th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
- link left_hand_1_4: geometry collision mesh filename=package://friday_description/meshes/FM26B/visual/left_hand_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; collision mesh filename=package://friday_description/meshes/FM26B/visual/tactile_th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
- link left_hand_2_2: geometry collision mesh filename=package://friday_description/meshes/FM26B/visual/left_hand_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; collision mesh filename=package://friday_description/meshes/FM26B/visual/tactile_mc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
- link left_hand_2_3: geometry collision mesh filename=package://friday_description/meshes/FM26B/visual/left_hand_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; collision mesh filename=package://friday_description/meshes/FM26B/visual/tactile_pi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
- link left_hand_2_4: geometry collision mesh filename=package://friday_description/meshes/FM26B/visual/left_hand_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; collision mesh filename=package://friday_description/meshes/FM26B/visual/tactile_di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
- link left_hand_3_2: geometry collision mesh filename=package://friday_description/meshes/FM26B/visual/left_hand_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; collision mesh filename=package://friday_description/meshes/FM26B/visual/tactile_mc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
- link left_hand_3_3: geometry collision mesh filename=package://friday_description/meshes/FM26B/visual/left_hand_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; collision mesh filename=package://friday_description/meshes/FM26B/visual/tactile_pi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
- link left_hand_3_4: geometry collision mesh filename=package://friday_description/meshes/FM26B/visual/left_hand_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; collision mesh filename=package://friday_description/meshes/FM26B/visual/tactile_di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
- link left_hand_4_2: geometry collision mesh filename=package://friday_description/meshes/FM26B/visual/left_hand_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; collision mesh filename=package://friday_description/meshes/FM26B/visual/tactile_mc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
- link left_hand_4_3: geometry collision mesh filename=package://friday_description/meshes/FM26B/visual/left_hand_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; collision mesh filename=package://friday_description/meshes/FM26B/visual/tactile_pi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
- link left_hand_4_4: geometry collision mesh filename=package://friday_description/meshes/FM26B/visual/left_hand_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; collision mesh filename=package://friday_description/meshes/FM26B/visual/tactile_di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
- link left_hand_5_2: geometry collision mesh filename=package://friday_description/meshes/FM26B/visual/left_hand_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; collision mesh filename=package://friday_description/meshes/FM26B/visual/tactile_mc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
- link left_hand_5_3: geometry collision mesh filename=package://friday_description/meshes/FM26B/visual/left_hand_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; collision mesh filename=package://friday_description/meshes/FM26B/visual/tactile_pi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
- link left_hand_5_4: geometry collision mesh filename=package://friday_description/meshes/FM26B/visual/left_hand_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; collision mesh filename=package://friday_description/meshes/FM26B/visual/tactile_di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
- link right_arm_7: geometry collision mesh filename=package://friday_description/meshes/FM26B/visual/right_arm_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; collision mesh filename=package://friday_description/meshes/FM26B/visual/right_wris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
- link right_hand_1_2: geometry collision mesh filename=package://friday_description/meshes/FM26B/visual/right_hand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; collision mesh filename=package://friday_description/meshes/FM26B/visual/tactile_th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
- link right_hand_1_3: geometry collision mesh filename=package://friday_description/meshes/FM26B/visual/right_hand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; collision mesh filename=package://friday_description/meshes/FM26B/visual/tactile_th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
- link right_hand_1_4: geometry collision mesh filename=package://friday_description/meshes/FM26B/visual/right_hand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; collision mesh filename=package://friday_description/meshes/FM26B/visual/tactile_th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
- link right_hand_2_2: geometry collision mesh filename=package://friday_description/meshes/FM26B/visual/right_hand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; collision mesh filename=package://friday_description/meshes/FM26B/visual/tactile_mc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
- link right_hand_2_3: geometry collision mesh filename=package://friday_description/meshes/FM26B/visual/right_hand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; collision mesh filename=package://friday_description/meshes/FM26B/visual/tactile_pi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
- link right_hand_2_4: geometry collision mesh filename=package://friday_description/meshes/FM26B/visual/right_hand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; collision mesh filename=package://friday_description/meshes/FM26B/visual/tactile_di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
- link right_hand_3_2: geometry collision mesh filename=package://friday_description/meshes/FM26B/visual/right_hand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; collision mesh filename=package://friday_description/meshes/FM26B/visual/tactile_mc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
- link right_hand_3_3: geometry collision mesh filename=package://friday_description/meshes/FM26B/visual/right_hand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; collision mesh filename=package://friday_description/meshes/FM26B/visual/tactile_pi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
- link right_hand_3_4: geometry collision mesh filename=package://friday_description/meshes/FM26B/visual/right_hand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; collision mesh filename=package://friday_description/meshes/FM26B/visual/tactile_di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
- link right_hand_4_2: geometry collision mesh filename=package://friday_description/meshes/FM26B/visual/right_hand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; collision mesh filename=package://friday_description/meshes/FM26B/visual/tactile_mc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
- link right_hand_4_3: geometry collision mesh filename=package://friday_description/meshes/FM26B/visual/right_hand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; collision mesh filename=package://friday_description/meshes/FM26B/visual/tactile_pi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
- link right_hand_4_4: geometry collision mesh filename=package://friday_description/meshes/FM26B/visual/right_hand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; collision mesh filename=package://friday_description/meshes/FM26B/visual/tactile_di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
- link right_hand_5_2: geometry collision mesh filename=package://friday_description/meshes/FM26B/visual/right_hand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; collision mesh filename=package://friday_description/meshes/FM26B/visual/tactile_mc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
- link right_hand_5_3: geometry collision mesh filename=package://friday_description/meshes/FM26B/visual/right_hand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; collision mesh filename=package://friday_description/meshes/FM26B/visual/tactile_pi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
- link right_hand_5_4: geometry collision mesh filename=package://friday_description/meshes/FM26B/visual/right_hand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; collision mesh filename=package://friday_description/meshes/FM26B/visual/tactile_di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
Joints:
- joint waist_1: origin xyz=0.0 0.0 0.14 rpy=0.0 0.0 0.0 -> xyz=0.0 0.0 0.144 rpy=0.0 0.0 0.0

Commit message: chore: sync friday_ros2 from holiday
GitOrigin-RevId: bcafb25a97730be2d5050c7c52102cb20f450a23

File: friday_description/urdf/FM26B.urdf (robot description, URDF)
Before this commit: robot FM26B, 90 links, 89 joints
Joints:
- joint head_1: limit lower=-0.855 upper=0.3316 effort=10.0 velocity=35.19 -> lower=-0.5235 upper=0.698 effort=10.0 velocity=35.19
- joint head_stereo: origin xyz=0.1106 0.03 -0.0311 rpy=-1.710423 -5.551115123125783e-17 -1.5707959999999999 -> xyz=0.1114557968 0.0289043036 -0.0289377725 rpy=-1.708320651315582 -0.0012623822334294434 -1.5661418619152416

Commit message: chore: sync friday_ros2 from holiday
GitOrigin-RevId: 97c730cec9f49e33f23578b594574daa66a60c9d

File: friday_description/urdf/FM26B.urdf (robot description, URDF)
Before this commit: robot FM26B, 90 links, 89 joints
Links:
- link left_arm_7: mass 0.297000291735 -> 0.362874
- link right_arm_7: mass 0.300897291735 -> 0.362874
Joints:
- joint head_1: limit lower=-0.5235 upper=0.698 effort=10.0 velocity=35.19 -> lower=-0.5235 upper=0.698 effort=10.0 velocity=35.185837
- joint head_2: limit lower=-0.2792 upper=0.2792 effort=10.0 velocity=35.19 -> lower=-0.2792 upper=0.2792 effort=10.0 velocity=35.185837
- joint head_3: limit lower=-0.965 upper=0.965 effort=10.0 velocity=35.19 -> lower=-0.965 upper=0.965 effort=10.0 velocity=35.185837
- joint left_arm_1: limit lower=-2.268 upper=0.7853 effort=130.0 velocity=11.96 -> lower=-2.268 upper=0.7853 effort=130.0 velocity=11.963184
- joint left_arm_2: limit lower=-0.1 upper=2.97 effort=130.0 velocity=11.96 -> lower=-0.1 upper=2.97 effort=130.0 velocity=11.963184
- joint left_arm_3: limit lower=-1.38 upper=1.38 effort=68.3 velocity=11.47 -> lower=-1.38 upper=1.38 effort=68.3 velocity=11.470584
- joint left_arm_4: limit lower=-2.02 upper=0.0 effort=71.7 velocity=3.95 -> lower=-2.02 upper=0.0 effort=71.7 velocity=8.701034
- joint left_arm_5: limit lower=-1.5708 upper=1.5708 effort=12.5 velocity=30.93 -> lower=-1.5708 upper=1.5708 effort=12.5 velocity=35.185837
- joint left_arm_6: limit lower=-0.785398 upper=0.785398 effort=12.5 velocity=35.19 -> lower=-0.785398 upper=0.785398 effort=12.5 velocity=35.185837
- joint left_arm_7: limit lower=-0.7155 upper=0.7155 effort=12.5 velocity=35.19 -> lower=-0.7155 upper=0.7155 effort=12.5 velocity=35.185837
- joint left_hand_1_1: origin xyz=0.0263009 -0.05775 -0.0944413 rpy=-2.61799 0.0 -1.5707999999999998 -> xyz=0.0263009 -0.05775 -0.1244413 rpy=-2.61799 0.0 -1.5707999999999998
- joint left_hand_2_1: origin xyz=0.0392 -0.05375 -0.151 rpy=-1.5707999999999998 0.0349066 -3.14159 -> xyz=0.0392 -0.05375 -0.181 rpy=-1.5707999999999998 0.0349066 -3.14159
- joint left_hand_3_1: origin xyz=0.0182 -0.05375 -0.1535 rpy=-1.5707999999999998 0.0 -3.14159 -> xyz=0.0182 -0.05375 -0.1835 rpy=-1.5707999999999998 0.0 -3.14159
- joint left_hand_4_1: origin xyz=-0.0028 -0.05375 -0.1495 rpy=-1.5708 -0.0349066 -3.14159 -> xyz=-0.0028 -0.05375 -0.1795 rpy=-1.5708 -0.0349066 -3.14159
- joint left_hand_5_1: origin xyz=-0.0238 -0.05375 -0.1455 rpy=-1.5707999999999998 -0.06981319999999998 -3.14159 -> xyz=-0.0238 -0.05375 -0.1755 rpy=-1.5707999999999998 -0.06981319999999998 -3.14159
- joint left_wrist_cam: origin xyz=-0.00975 -0.063081 -0.071184 rpy=2.3561945 0.0 0.0 -> xyz=-0.00975 -0.063081 -0.101184 rpy=2.3561945 0.0 0.0
- joint right_arm_1: limit lower=-2.268 upper=0.7853 effort=130.0 velocity=11.96 -> lower=-2.268 upper=0.7853 effort=130.0 velocity=11.963184
- joint right_arm_2: limit lower=-2.97 upper=0.1 effort=130.0 velocity=11.96 -> lower=-2.97 upper=0.1 effort=130.0 velocity=11.963184
- joint right_arm_3: limit lower=-1.38 upper=1.38 effort=68.3 velocity=11.47 -> lower=-1.38 upper=1.38 effort=68.3 velocity=11.470584
- joint right_arm_4: limit lower=-2.02 upper=0.0 effort=71.7 velocity=3.95 -> lower=-2.02 upper=0.0 effort=71.7 velocity=8.701034
- joint right_arm_5: limit lower=-1.5708 upper=1.5708 effort=12.5 velocity=30.93 -> lower=-1.5708 upper=1.5708 effort=12.5 velocity=35.185837
- joint right_arm_6: limit lower=-0.785398 upper=0.785398 effort=12.5 velocity=35.19 -> lower=-0.785398 upper=0.785398 effort=12.5 velocity=35.185837
- joint right_arm_7: limit lower=-0.7155 upper=0.7155 effort=12.5 velocity=35.19 -> lower=-0.7155 upper=0.7155 effort=12.5 velocity=35.185837
- joint right_hand_1_1: origin xyz=0.0263009 0.05775 -0.0944413 rpy=-0.523599 4.0000225354219765e-12 1.5708 -> xyz=0.0263009 0.05775 -0.1244413 rpy=-0.523599 4.0000225354219765e-12 1.5708
- joint right_hand_2_1: origin xyz=0.0392 0.05375 -0.151 rpy=1.5707999999999998 -0.0349066 -1.000000715683979e-12 -> xyz=0.0392 0.05375 -0.181 rpy=1.5707999999999998 -0.0349066 -1.000000715683979e-12
- joint right_hand_3_1: origin xyz=0.0182 0.05375 -0.1535 rpy=1.5707999999999998 9.999999999999998e-13 -1e-12 -> xyz=0.0182 0.05375 -0.1835 rpy=1.5707999999999998 9.999999999999998e-13 -1e-12
- joint right_hand_4_1: origin xyz=-0.0028 0.05375 -0.1495 rpy=1.5708 0.0349066 -9.99993772560508e-13 -> xyz=-0.0028 0.05375 -0.1795 rpy=1.5708 0.0349066 -9.99993772560508e-13
- joint right_hand_5_1: origin xyz=-0.0238 0.05375 -0.1455 rpy=1.5707999999999998 0.0698132 -1.000006048656765e-12 -> xyz=-0.0238 0.05375 -0.1755 rpy=1.5707999999999998 0.0698132 -1.000006048656765e-12
- joint right_wrist_cam: origin xyz=-0.00975 0.063081 -0.071184 rpy=2.3561945 3.308722450212111e-24 3.1415926071795868 -> xyz=-0.00975 0.063081 -0.101184 rpy=2.3561945 3.308722450212111e-24 3.1415926071795868
- joint waist_1: limit lower=-5.4978 upper=5.4978 effort=530.4 velocity=2.93 -> lower=-5.4978 upper=5.4978 effort=530.4 velocity=2.932153
- joint waist_2: limit lower=-1.5708 upper=0.174533 effort=837.2 velocity=1.86 -> lower=-1.5708 upper=0.174533 effort=837.2 velocity=1.857637
- joint waist_3: limit lower=-0.174533 upper=2.618 effort=837.2 velocity=1.86 -> lower=-0.174533 upper=2.618 effort=837.2 velocity=1.857637
- joint waist_4: limit lower=-1.8326 upper=1.0472 effort=837.2 velocity=1.86 -> lower=-1.8326 upper=1.0472 effort=837.2 velocity=1.857637
- joint waist_5: limit lower=-5.4978 upper=5.4978 effort=450.8 velocity=3.45 -> lower=-5.4978 upper=5.4978 effort=450.8 velocity=3.449592
